Commit message: fix minor bugs

File: dh_ag95_description/urdf/dh_ag95_macro.xacro (robot description, xacro)
@@ -7,8 +7,8 @@
     *origin"
   >
-    <xacro:property name="lower_limit" value="0" />
+    <xacro:property name="lower_limit" value="0.0" />
     <xacro:property name="upper_limit" value="0.93" />
     <xacro:property name="max_effort" value="50.0" />
-    <xacro:property name="max_velocity" value="2.0" />
+    <xacro:property name="max_velocity" value="2.1" />
     <!-- fingers links macros -->
     <xacro:macro name="outer_knuckle" params="prefix fingerprefix">

File: dh_gripper_driver/urdf/dh_ag95.ros2_control.xacro (robot description, xacro)
@@ -6,5 +6,5 @@
                 <xacro:if value="${use_mock_hardware}">
                     <plugin>mock_components/GenericSystem</plugin>
-                    <param name="fake_sensor_commands">${fake_sensor_commands}</param>
+                    <param name="mock_sensor_commands">${mock_sensor_commands}</param>
                     <param name="state_following_offset">0.0</param>
                 </xacro:if>

Commit message: added grasp link to urdf

File: dh_ag95_description/urdf/dh_ag95_macro.xacro (robot description, xacro)
@@ -4,4 +4,5 @@
     params="
     prefix
+    grasp_link_offset:=0.19
     parent
     *origin"
@@ -263,4 +264,10 @@
       <child link="${prefix}ag95_body" />
     </joint>
+    <link name="${prefix}grasp_link"/>
+    <joint name="${prefix}grasp_joint" type="fixed">
+      <parent link="${prefix}ag95_base_link" />
+      <child link="${prefix}grasp_link" />
+      <origin xyz="0.0 0.0 ${grasp_link_offset}" rpy="${pi/2} ${-pi/2} 0" />
+    </joint>
     <!-- left finger -->
     <xacro:finger_links prefix="${prefix}" fingerprefix="left" />
